Commit message: Add files via upload

File: urdf/my_robot_arm.urdf (robot description, URDF)
Before this commit: robot my_robot_arm, 2 links, 1 joints
Links:
- added link Elbow_Joint; visual cylinder length=0.1 radius=0.1
- added link Shoulder_Joint; visual cylinder length=0.1 radius=0.1
- added link Shoulder_Joint_Link; visual box size=0.1 0.4 0.1
- added link Waist_joint; visual cylinder length=0.20 radius=0.1
- link Robot_stand: mass 0.7 -> None; geometry visual box size=0.2 0.2 0.5
Joints:
- added joint Link01__Elbow_Joint: type revolute, parent Shoulder_Joint_Link, child Elbow_Joint, origin xyz=0 0.3 0 rpy=0 0 0, axis 0 0 1, limit lower=-3.14 upper=3.14 effort=1000.0 velocity=0.5
- added joint Robot_stand__Waist_Joint: type revolute, parent Robot_stand, child Waist_joint, origin xyz=0 0 0.25 rpy=0 0 0, axis 0 0 1, limit lower=-3.14 upper=3.14 effort=1000.0 velocity=0.5
- added joint Shoulder_Joint__Link01: type fixed, parent Shoulder_Joint, child Shoulder_Joint_Link, origin xyz=0 0.2 0 rpy=0 0 0
- added joint Waist_Joint__Shoulder_Joint: type revolute, parent Waist_joint, child Shoulder_Joint, origin xyz=0 0 0.20 rpy=1.57 0 0, axis 0 0 1, limit lower=-3.14 upper=3.14 effort=1000.0 velocity=0.5

Commit message: Ended with end effector
it is a simple showcase for urdf code that presents a manipulator
To Do: Adding collisions and inertia

File: urdf/my_robot_arm.urdf (robot description, URDF)
Before this commit: robot my_robot_arm_description, 6 links, 5 joints
Links:
- added link Elbow_Joint_Link; visual box size=0.1 0.3 0.1
- added link Wrist_Joint; visual cylinder length=0.1 radius=0.1
- added link Wrist_Joint_Link; visual box size=0.1 0.1 0.1
Joints:
- added joint Elbow_Joint__Link02: type fixed, parent Elbow_Joint, child Elbow_Joint_Link, origin xyz=0 0.20 0 rpy=0 0 0
- added joint Link02__Wrist_Joint: type revolute, parent Elbow_Joint_Link, child Wrist_Joint, origin xyz=0 0.20 0 rpy=0 0 0, axis 0 0 1, limit lower=-3.14 upper=3.14 effort=1000.0 velocity=0.5
- added joint Wrist_Joint__End_Effector: type fixed, parent Wrist_Joint, child Wrist_Joint_Link, origin xyz=0 0.1 0 rpy=0 0 0
- joint Link01__Elbow_Joint: origin xyz=0 0.3 0 rpy=0 0 0 -> xyz=0 0.25 0 rpy=0 0 0
- joint Shoulder_Joint__Link01: origin xyz=0 0.2 0 rpy=0 0 0 -> xyz=0 0.25 0 rpy=0 0 0
